File: HARDWARE/FUTBOLISTA.kicad_pcb (KiCad board)
At the start: 2 copper layers, 16 parts, among them J1 Screw_Terminal_01x02, J2 Screw_Terminal_01x02, J3 Conn_01x08_Socket, J4 ENTRADA, J5 Conn_01x08_Socket, U1 ESP32_DEVKITC, U2 L7805

Commit message: Add files via upload
Parts:
- removed J1, J2: Screw_Terminal_01x02, EESTN5:BORNERA2
- moved LLAVE1 19.9 mm to (40.5, 41.7), turned to 90 degrees
- moved J4 5.40 mm to (31.8, 34.5), turned to -90 degrees
- moved REF** 3.65 mm to (27.2, 26.6)
- moved REF** 3.65 mm to (77.5, 26.6)
Connections:
- U1 pad 10: unconnected-(U1-IO26-Pad10) -> RPWM_2
- U1 pad 11: RPWM_2 -> LPWM_2
- U1 pad 12: LPWM_2 -> unconnected-(U1-IO14-Pad12)
Routing:
- net VCC: track 104.0 -> 39.6 mm
- net Net-(J4-Pin_2): track 14.5 -> 8.70 mm
- net RPWM_2: track 8.10 -> 10.4 mm
- net LPWM_2: track 8.10 -> 9.97 mm
