File: HARDWARE/FUTBOLISTA.kicad_sch (KiCad schematic)
At the start: 12 parts, among them J1 Screw_Terminal_01x02, J2 Screw_Terminal_01x02, J3 Conn_01x08_Socket, J4 ENTRADA, J5 Conn_01x08_Socket, U1 ESP32_DEVKITC, U2 L7805

Commit message: Add files via upload
Parts:
- removed J1, J2: Screw_Terminal_01x02, EESTN5:BORNERA2, symbol Connector:Screw_Terminal_01x02
Connections:
- net LPWM_2: now also U1.11 (IO27); no longer U1.12 (IO14)
- net RPWM_2: now also U1.10 (IO26); no longer U1.11 (IO27)
